File: hardware/eduquencer/dac.kicad_sch (KiCad schematic)
At the start: 16 parts, among them IC5 DAC80501MDGST, IC6 OPA172IDR, J14 Out A

Commit message: Hardware: assign all footprints
Parts:
- C21, C22, C23, C24, C25, C26: footprint Capacitor_SMD:C_0603_1608Metric -> Capacitor_SMD:C_0603_1608Metric_Pad1.08x0.95mm_HandSolder
- IC5: footprint SOP50P490X110-10N -> DAC80501MDGST:SOP50P490X110-10N
- IC6: footprint SOIC127P600X175-8N -> OPA172IDR:SOIC127P600X175-8N
- R54, R57: footprint (none) -> Resistor_SMD:R_0603_1608Metric_Pad0.98x0.95mm_HandSolder
- R55, R56, R58, R59, R60: footprint Resistor_SMD:R_0603_1608Metric -> Resistor_SMD:R_0603_1608Metric_Pad0.98x0.95mm_HandSolder
Changed lines of the file:
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@@
       (effects (font (size 1.27 1.27)) (justify right))
     )
-    (property "Footprint" "Capacitor_SMD:C_0603_1608Metric" (id 2) (at 51.1048 36.83 0)
+    (property "Footprint" "Capacitor_SMD:C_0603_1608Metric_Pad1.08x0.95mm_HandSolder" (id 2) (at 51.1048 36.83 0)
       (effects (font (size 1.27 1.27)) hide)
     )
@@
       (effects (font (size 1.27 1.27)) (justify left))
     )
-    (property "Footprint" "Capacitor_SMD:C_0603_1608Metric" (id 2) (at 63.1952 44.45 0)
+    (property "Footprint" "Capacitor_SMD:C_0603_1608Metric_Pad1.08x0.95mm_HandSolder" (id 2) (at 63.1952 44.45 0)
       (effects (font (size 1.27 1.27)) hide)
     )
@@
       (effects (font (size 1.27 1.27)) (justify right))
     )
-    (property "Footprint" "Capacitor_SMD:C_0603_1608Metric" (id 2) (at 79.6798 36.83 0)
+    (property "Footprint" "Capacitor_SMD:C_0603_1608Metric_Pad1.08x0.95mm_HandSolder" (id 2) (at 79.6798 36.83 0)
       (effects (font (size 1.27 1.27)) hide)
     )
@@
       (effects (font (size 1.27 1.27)) (justify right))
     )
-    (property "Footprint" "Resistor_SMD:R_0603_1608Metric" (id 2) (at 53.848 101.6 90)
+    (property "Footprint" "Resistor_SMD:R_0603_1608Metric_Pad0.98x0.95mm_HandSolder" (id 2) (at 53.848 101.6 90)
       (effects (font (size 1.27 1.27)) hide)
     )
@@
     (property "Reference" "R58" (id 0) (at 129.54 87.8078 90))
     (property "Value" "33k" (id 1) (at 129.54 85.4964 90))
-    (property "Footprint" "Resistor_SMD:R_0603_1608Metric" (id 2) (at 129.54 80.772 90)
+    (property "Footprint" "Resistor_SMD:R_0603_1608Metric_Pad0.98x0.95mm_HandSolder" (id 2) (at 129.54 80.772 90)
       (effects (font (size 1.27 1.27)) hide)
     )
@@
       (effects (font (size 1.27 1.27)) (justify left))
     )
-    (property "Footprint" "Resistor_SMD:R_0603_1608Metric" (id 2) (at 50.292 86.36 90)
+    (property "Footprint" "Resistor_SMD:R_0603_1608Metric_Pad0.98x0.95mm_HandSolder" (id 2) (at 50.292 86.36 90)
       (effects (font (size 1.27 1.27)) hide)
     )
@@
     (property "Reference" "R60" (id 0) (at 208.28 90.3478 90))
     (property "Value" "1k" (id 1) (at 208.28 88.0364 90))
-    (property "Footprint" "Resistor_SMD:R_0603_1608Metric" (id 2) (at 208.28 83.312 90)
+    (property "Footprint" "Resistor_SMD:R_0603_1608Metric_Pad0.98x0.95mm_HandSolder" (id 2) (at 208.28 83.312 90)
       (effects (font (size 1.27 1.27)) hide)
     )
@@
     (property "Reference" "R59" (id 0) (at 182.88 118.2878 90))
     (property "Value" "180k" (id 1) (at 182.88 115.9764 90))
-    (property "Footprint" "Resistor_SMD:R_0603_1608Metric" (id 2) (at 182.88 111.252 90)
+    (property "Footprint" "Resistor_SMD:R_0603_1608Metric_Pad0.98x0.95mm_HandSolder" (id 2) (at 182.88 111.252 90)
       (effects (font (size 1.27 1.27)) hide)
     )
@@
       (effects (font (size 1.27 1.27)) (justify right))
     )
-    (property "Footprint" "Capacitor_SMD:C_0603_1608Metric" (id 2) (at 99.3648 36.83 0)
+    (property "Footprint" "Capacitor_SMD:C_0603_1608Metric_Pad1.08x0.95mm_HandSolder" (id 2) (at 99.3648 36.83 0)
       (effects (font (size 1.27 1.27)) hide)
     )
@@
       (effects (font (size 1.27 1.27)) (justify right))
     )
-    (property "Footprint" "Capacitor_SMD:C_0603_1608Metric" (id 2) (at 115.8748 36.83 0)
+    (property "Footprint" "Capacitor_SMD:C_0603_1608Metric_Pad1.08x0.95mm_HandSolder" (id 2) (at 115.8748 36.83 0)
       (effects (font (size 1.27 1.27)) hide)
     )
@@
       (effects (font (size 1.27 1.27)) (justify right))
     )
-    (property "Footprint" "Capacitor_SMD:C_0603_1608Metric" (id 2) (at 168.91 100.6348 0)
+    (property "Footprint" "Capacitor_SMD:C_0603_1608Metric_Pad1.08x0.95mm_HandSolder" (id 2) (at 168.91 100.6348 0)
       (effects (font (size 1.27 1.27)) hide)
     )
@@
     (property "Reference" "R54" (id 0) (at 49.53 156.21 90))
     (property "Value" "4k7" (id 1) (at 49.53 158.75 90))
-    (property "Footprint" "" (id 2) (at 49.53 152.4 0)
+    (property "Footprint" "Resistor_SMD:R_0603_1608Metric_Pad0.98x0.95mm_HandSolder" (id 2) (at 49.53 152.4 0)
       (effects (font (size 1.27 1.27)) hide)
     )
@@
       (effects (font (size 1.27 1.27)) (justify left))
     )
-    (property "Footprint" "" (id 2) (at 110.49 144.78 0)
+    (property "Footprint" "Resistor_SMD:R_0603_1608Metric_Pad0.98x0.95mm_HandSolder" (id 2) (at 110.49 144.78 0)
       (effects (font (size 1.27 1.27)) hide)
     )
@@
     (property "Reference" "IC5" (id 0) (at 74.93 134.62 0))
     (property "Value" "DAC80501MDGST" (id 1) (at 74.93 137.16 0))
-    (property "Footprint" "SOP50P490X110-10N" (id 2) (at 88.9 139.7 0)
+    (property "Footprint" "DAC80501MDGST:SOP50P490X110-10N" (id 2) (at 88.9 139.7 0)
       (effects (font (size 1.27 1.27)) (justify left) hide)
     )
@@
     (property "Reference" "IC6" (id 0) (at 166.37 72.39 0))
     (property "Value" "OPA172IDR" (id 1) (at 166.37 74.93 0))
-    (property "Footprint" "SOIC127P600X175-8N" (id 2) (at 176.53 77.47 0)
-      (effects (font (size 1.27 1.27)) (justify left) hide)
-    )
+    (property "Footprint" "OPA172IDR:SOIC127P600X175-8N" (id 2) (at 176.53 77.47 0)
+      (effects (font (size 1.27 1.27)) (justify left) hide)
+    )
